File: ribv6.kicad_pcb (KiCad board)
At the start: 2 copper layers, 67.3 x 75 mm, 11 parts, among them J1 Conn_01x19, J2 Conn_01x19, J3 Conn_01x19, J4 Conn_01x19, J5 Conn_01x19, J6 Conn_01x19, J7 Conn_01x19, J8 Conn_01x19, U1 ESP32-DEVKITC-32D

Commit message: Add schematic and PCB #20
Parts:
- removed svg2mod (x2): G***, outline:rib_outline
- added D1: LED_Small, LED_SMD:LED_0805_2012Metric, F.Cu at (163.5, 92.2)
- added D2: LED_Small, LED_SMD:LED_0805_2012Metric, F.Cu at (87.5, 92.5)
- added D3: LED_Small, LED_SMD:LED_0805_2012Metric, F.Cu at (161.7, 52.1)
- added D4: LED_Small, LED_SMD:LED_0805_2012Metric, F.Cu at (161.7, 64.3)
- added D5: LED_Small, LED_SMD:LED_0805_2012Metric, F.Cu at (161.7, 68.4)
- added D6: LED_Small, LED_SMD:LED_0805_2012Metric, F.Cu at (161.7, 56.2)
- added D7: LED_Small, LED_SMD:LED_0805_2012Metric, F.Cu at (161.7, 60.2)
- added D8: LED_Small, LED_SMD:LED_0805_2012Metric, F.Cu at (112.8, 158.0)
- added F1: Fuse, 3557-2:3557-2, F.Cu at (149.9, 90.8)
- added F2: Fuse, 3557-2:3557-2, F.Cu at (101.2, 90.8)
- added F3: Fuse, 3557-2:3557-2, F.Cu at (88.2, 60.4)
- added F4: Fuse, 3557-2:3557-2, F.Cu at (129.5, 71.1)
- added F5: Fuse, 3557-2:3557-2, F.Cu at (149.7, 71.1)
- added J10: Conn_01x19, Connector_PinHeader_2.54mm:PinHeader_1x19_P2.54mm_Vertical, F.Cu at (97.7, 96.3)
- added J11: Conn_01x01_Male, P315100rH:P315100rH, F.Cu at (100.6, 59.2)
- added J12: Conn_01x01_Male, MountingHole:MountingHole_3.5mm_Pad, F.Cu at (126.5, 39.5)
- added J13: Conn_01x19, Connector_PinHeader_2.54mm:PinHeader_1x19_P2.54mm_Vertical, F.Cu at (102.7, 96.3)
- added J14: Conn_02x04_Odd_Even, Connector_PinSocket_2.54mm:PinSocket_2x04_P2.54mm_Vertical, F.Cu at (153.5, 157.3)
- added J15: Conn_02x04_Odd_Even, Connector_PinSocket_2.54mm:PinSocket_2x04_P2.54mm_Vertical, F.Cu at (153.5, 149.6)
- added J16: Conn_01x19, Connector_PinHeader_2.54mm:PinHeader_1x19_P2.54mm_Vertical, F.Cu at (107.8, 96.3)
- added J19: Conn_01x19, Connector_PinHeader_2.54mm:PinHeader_1x19_P2.54mm_Vertical, F.Cu at (135.8, 96.3)
- added J20: Conn_01x19, Connector_PinHeader_2.54mm:PinHeader_1x19_P2.54mm_Vertical, F.Cu at (143.4, 96.3)
- added J21: Conn_01x19, Connector_PinHeader_2.54mm:PinHeader_1x19_P2.54mm_Vertical, F.Cu at (148.5, 96.3)
- added J22: Conn_01x06, Connector_PinHeader_2.54mm:PinHeader_1x06_P2.54mm_Vertical, F.Cu at (102.7, 144.6)
- added J23: Conn_02x06_Odd_Even, Connector_PinSocket_2.54mm:PinSocket_2x06_P2.54mm_Vertical, F.Cu at (100.2, 144.6)
- added J24: Conn_01x01_Male, MountingHole:MountingHole_3.5mm_Pad, F.Cu at (152.8, 39.6)
- added J25: Conn_01x06, wiichuck:CONN_WII, F.Cu at (140.1, 39.0)
- added J26: Conn_01x01_Male, P315100rH:P315100rH, F.Cu at (114.5, 59.2)
- added J9: Conn_01x03, Connector_PinHeader_2.54mm:PinHeader_1x03_P2.54mm_Vertical, F.Cu at (113.5, 85.2)
- added Q1: BSS138, Package_TO_SOT_SMD:SOT-23, F.Cu at (163.5, 89.2)
- added Q10: BSS138, Package_TO_SOT_SMD:SOT-23, F.Cu at (130.4, 112.2)
- added Q11: BSS138, Package_TO_SOT_SMD:SOT-23, F.Cu at (130.4, 115.6)
- added Q12: BSS138, Package_TO_SOT_SMD:SOT-23, F.Cu at (130.5, 119.7)
- added Q13: BSS138, Package_TO_SOT_SMD:SOT-23, F.Cu at (118.8, 125.3)
- added Q14: BSS138, Package_TO_SOT_SMD:SOT-23, F.Cu at (118.8, 117.7)
- added Q15: BSS138, Package_TO_SOT_SMD:SOT-23, F.Cu at (130.5, 123.2)
- added Q2: BSS138, Package_TO_SOT_SMD:SOT-23, F.Cu at (124.6, 56.3)
- added Q3: BSS138, Package_TO_SOT_SMD:SOT-23, F.Cu at (117.6, 76.2)
- added Q4: BSS138, Package_TO_SOT_SMD:SOT-23, F.Cu at (113.5, 89.2)
- added Q5: BSS138, Package_TO_SOT_SMD:SOT-23, F.Cu at (128.0, 77.0)
- added Q6: BSS138, Package_TO_SOT_SMD:SOT-23, F.Cu at (132.5, 89.2)
- added Q7: BSS138, Package_TO_SOT_SMD:SOT-23, F.Cu at (87.5, 89.2)
- added Q8: BSS138, Package_TO_SOT_SMD:SOT-23, F.Cu at (130.4, 108.7)
- added Q9: BSS138, Package_TO_SOT_SMD:SOT-23, F.Cu at (130.4, 105.1)
- added R1: R_Small, Resistor_SMD:R_0603_1608Metric, F.Cu at (160.8, 92.2)
- added R10: R_Small, Resistor_SMD:R_0603_1608Metric, F.Cu at (132.0, 76.7)
- added R11: R_Small, Resistor_SMD:R_0603_1608Metric, F.Cu at (130.5, 76.7)
- added R12: R_Small, Resistor_SMD:R_0603_1608Metric, F.Cu at (136.6, 89.0)
- added R13: R_Small, Resistor_SMD:R_0603_1608Metric, F.Cu at (135.1, 89.0)
- added R14: R_Small, Resistor_SMD:R_0603_1608Metric, F.Cu at (90.2, 92.2)
- added R15: R_Small, Resistor_SMD:R_0603_1608Metric, F.Cu at (90.2, 89.0)
- added R16: 330, Resistor_SMD:R_0603_1608Metric, F.Cu at (87.8, 94.5)
- added R17: 10k, Resistor_SMD:R_0603_1608Metric, F.Cu at (133.0, 108.9)
- added R18: 10k, Resistor_SMD:R_0603_1608Metric, F.Cu at (133.0, 105.4)
- added R19: 10k, Resistor_SMD:R_0603_1608Metric, F.Cu at (133.0, 112.4)
- added R2: R_Small, Resistor_SMD:R_0603_1608Metric, F.Cu at (129.5, 56.8)
- added R20: 10k, Resistor_SMD:R_0603_1608Metric, F.Cu at (133.0, 115.9)
- added R21: 10k, Resistor_SMD:R_0603_1608Metric, F.Cu at (133.0, 119.9)
- added R22: 10k, Resistor_SMD:R_0603_1608Metric, F.Cu at (127.9, 108.9)
- added R23: 10k, Resistor_SMD:R_0603_1608Metric, F.Cu at (127.9, 105.4)
- added R24: 10k, Resistor_SMD:R_0603_1608Metric, F.Cu at (127.9, 112.4)
- added R25: 10k, Resistor_SMD:R_0603_1608Metric, F.Cu at (127.9, 115.9)
- added R26: 10k, Resistor_SMD:R_0603_1608Metric, F.Cu at (127.9, 120.0)
- added R27: 10k, Resistor_SMD:R_0603_1608Metric, F.Cu at (116.3, 125.0)
- added R28: 10k, Resistor_SMD:R_0603_1608Metric, F.Cu at (116.2, 117.4)
- added R29: 10k, Resistor_SMD:R_0603_1608Metric, F.Cu at (133.0, 123.4)
- added R3: R_Small, Resistor_SMD:R_0603_1608Metric, F.Cu at (127.2, 56.0)
- added R30: 10k, Resistor_SMD:R_0603_1608Metric, F.Cu at (121.3, 125.0)
- added R31: 10k, Resistor_SMD:R_0603_1608Metric, F.Cu at (121.3, 117.4)
- added R32: 10k, Resistor_SMD:R_0603_1608Metric, F.Cu at (127.9, 123.4)
- added R33: 330, Resistor_SMD:R_0603_1608Metric, F.Cu at (161.5, 66.1)
- added R34: R_Small, Resistor_SMD:R_0603_1608Metric, F.Cu at (161.5, 70.2)
- added R35: 330, Resistor_SMD:R_0603_1608Metric, F.Cu at (161.5, 53.9)
- added R36: 330, Resistor_SMD:R_0603_1608Metric, F.Cu at (161.6, 62.0)
- added R37: 330, Resistor_SMD:R_0603_1608Metric, F.Cu at (161.5, 58.0)
- added R38: 10k, Resistor_SMD:R_0603_1608Metric, F.Cu at (132.5, 99.0)
- added R39: 330, Resistor_SMD:R_0603_1608Metric, F.Cu at (112.8, 154.5)
- added R4: R_Small, Resistor_SMD:R_0603_1608Metric, F.Cu at (113.6, 76.5)
- added R5: R_Small, Resistor_SMD:R_0603_1608Metric, F.Cu at (115.1, 76.5)
- added R6: R_Small, Resistor_SMD:R_0603_1608Metric, F.Cu at (116.0, 89.0)
- added R7: R_Small, Resistor_SMD:R_0603_1608Metric, F.Cu at (117.5, 89.0)
- added R8: R_Small, Resistor_SMD:R_0603_1608Metric, F.Cu at (160.8, 89.0)
- added R9: 330, Resistor_SMD:R_0603_1608Metric, F.Cu at (163.2, 94.2)
- added U2: polulu-3784-D36V28F7, polulu-3784-dcdcreg:polulu-3784-D36V28F7, F.Cu at (143.5, 65.9)
- added U3: esp-devkit, esp-devkit:ESP-DEVKIT, F.Cu at (112.9, 142.0)
- added U4: DPDT_x2, GF-126-0327:GF-126-0327, F.Cu at (102.1, 65.3)
- J1: value Conn_01x19 -> Conn_01x03; footprint Connector_PinHeader_2.54mm:PinHeader_1x19_P2.54mm_Vertical -> Connector_PinHeader_2.54mm:PinHeader_1x03_P2.54mm_Vertical
- J2, J6: value Conn_01x19 -> Conn_01x02_Female; footprint Connector_PinHeader_2.54mm:PinHeader_1x19_P2.54mm_Vertical -> Connector_JST:JST_EH_B2B-EH-A_1x02_P2.50mm_Vertical
- J4, J8: value Conn_01x19 -> Conn_02x07_Odd_Even; footprint Connector_PinHeader_2.54mm:PinHeader_1x19_P2.54mm_Vertical -> Connector_PinSocket_2.54mm:PinSocket_2x07_P2.54mm_Vertical
- U1: value ESP32-DEVKITC-32D -> polulu-3784-D36V28F7; footprint MODULE_ESP32-DEVKITC-32D -> polulu-3784-dcdcreg:polulu-3784-D36V28F7
- moved J8 156.7 mm to (93.1, 82.4), turned to 90 degrees
- moved J7 151.0 mm to (100.2, 96.3)
- moved J6 128.4 mm to (113.5, 62.3)
- moved J2 121.4 mm to (113.5, 67.3)
- moved U1 90.7 mm to (125.2, 65.9)
- moved J1 70.1 mm to (137.7, 85.2), turned to 270 degrees
- moved J5 61.1 mm to (151.0, 96.3)
- moved J3 56.5 mm to (153.5, 96.3)
- moved J4 55.8 mm to (142.8, 82.4), turned to 90 degrees
Connections:
- J1 pad 2: Net-(J1-Pad2) -> UBEC1
- J1 pad 3: Net-(J1-Pad3) -> GND
- J2 pad 1: Net-(J2-Pad1) -> +BATT
- J2 pad 2: Net-(J2-Pad2) -> GND
- J3 pad 1: Net-(J3-Pad1) -> GND
- J3 pad 10: Net-(J3-Pad10) -> GND
- J3 pad 11: Net-(J3-Pad11) -> GND
- J3 pad 12: Net-(J3-Pad12) -> GND
- J3 pad 13: Net-(J3-Pad13) -> GND
- J3 pad 14: Net-(J3-Pad14) -> GND
- J3 pad 15: Net-(J3-Pad15) -> GND
- J3 pad 16: Net-(J3-Pad16) -> GND
- J3 pad 17: Net-(J3-Pad17) -> GND
- J3 pad 18: Net-(J3-Pad18) -> GND
- J3 pad 19: Net-(J3-Pad19) -> GND
- J3 pad 2: Net-(J3-Pad2) -> GND
- J3 pad 3: Net-(J3-Pad3) -> GND
- J3 pad 4: Net-(J3-Pad4) -> GND
- J3 pad 5: Net-(J3-Pad5) -> GND
- J3 pad 6: Net-(J3-Pad6) -> GND
- J3 pad 7: Net-(J3-Pad7) -> GND
- J3 pad 8: Net-(J3-Pad8) -> GND
- J3 pad 9: Net-(J3-Pad9) -> GND
- J4 pad 1: Net-(J4-Pad1) -> UBEC1
- J4 pad 10: Net-(J4-Pad10) -> Net-(F1-Pad1)
- J4 pad 12: Net-(J4-Pad12) -> Net-(F1-Pad1)
- J4 pad 13: Net-(J4-Pad13) -> +BATT
- J4 pad 14: Net-(J4-Pad14) -> Net-(F1-Pad1)
- J4 pad 2: Net-(J4-Pad2) -> Net-(F1-Pad1)
- J4 pad 4: Net-(J4-Pad4) -> Net-(F1-Pad1)
- J4 pad 5: Net-(J4-Pad5) -> +5V
- J4 pad 6: Net-(J4-Pad6) -> Net-(F1-Pad1)
- J4 pad 8: Net-(J4-Pad8) -> Net-(F1-Pad1)
- J4 pad 9: Net-(J4-Pad9) -> +3V3
- J5 pad 1: Net-(J5-Pad1) -> Rail1
- J5 pad 10: Net-(J5-Pad10) -> Rail1
- J5 pad 11: Net-(J5-Pad11) -> Rail1
- J5 pad 12: Net-(J5-Pad12) -> Rail1
- J5 pad 13: Net-(J5-Pad13) -> Rail1
- J5 pad 14: Net-(J5-Pad14) -> Rail1
- J5 pad 15: Net-(J5-Pad15) -> Rail1
- J5 pad 16: Net-(J5-Pad16) -> Rail1
- J5 pad 17: Net-(J5-Pad17) -> Rail1
- J5 pad 18: Net-(J5-Pad18) -> Rail1
- J5 pad 19: Net-(J5-Pad19) -> Rail1
- J5 pad 2: Net-(J5-Pad2) -> Rail1
- J5 pad 3: Net-(J5-Pad3) -> Rail1
- J5 pad 4: Net-(J5-Pad4) -> Rail1
- J5 pad 5: Net-(J5-Pad5) -> Rail1
- J5 pad 6: Net-(J5-Pad6) -> Rail1
- J5 pad 7: Net-(J5-Pad7) -> Rail1
- J5 pad 8: Net-(J5-Pad8) -> Rail1
- J5 pad 9: Net-(J5-Pad9) -> Rail1
- J6 pad 1: Net-(J6-Pad1) -> +BATT
- J6 pad 2: Net-(J6-Pad2) -> GND
- J7 pad 1: Net-(J7-Pad1) -> Rail2
- J7 pad 10: Net-(J7-Pad10) -> Rail2
- J7 pad 11: Net-(J7-Pad11) -> Rail2
- J7 pad 12: Net-(J7-Pad12) -> Rail2
- J7 pad 13: Net-(J7-Pad13) -> Rail2
- J7 pad 14: Net-(J7-Pad14) -> Rail2
- J7 pad 15: Net-(J7-Pad15) -> Rail2
- J7 pad 16: Net-(J7-Pad16) -> Rail2
- J7 pad 17: Net-(J7-Pad17) -> Rail2
- J7 pad 18: Net-(J7-Pad18) -> Rail2
- J7 pad 19: Net-(J7-Pad19) -> Rail2
- J7 pad 2: Net-(J7-Pad2) -> Rail2
- J7 pad 3: Net-(J7-Pad3) -> Rail2
- J7 pad 4: Net-(J7-Pad4) -> Rail2
- J7 pad 5: Net-(J7-Pad5) -> Rail2
- J7 pad 6: Net-(J7-Pad6) -> Rail2
- J7 pad 7: Net-(J7-Pad7) -> Rail2
- J7 pad 8: Net-(J7-Pad8) -> Rail2
- J7 pad 9: Net-(J7-Pad9) -> Rail2
- J8 pad 1: Net-(J8-Pad1) -> +BATT
- J8 pad 10: Net-(J8-Pad10) -> Net-(F2-Pad1)
- J8 pad 12: Net-(J8-Pad12) -> Net-(F2-Pad1)
- J8 pad 13: Net-(J8-Pad13) -> UBEC2
- J8 pad 14: Net-(J8-Pad14) -> Net-(F2-Pad1)
- J8 pad 2: Net-(J8-Pad2) -> Net-(F2-Pad1)
- J8 pad 4: Net-(J8-Pad4) -> Net-(F2-Pad1)
- J8 pad 5: Net-(J8-Pad5) -> +3V3
- J8 pad 6: Net-(J8-Pad6) -> Net-(F2-Pad1)
- J8 pad 8: Net-(J8-Pad8) -> Net-(F2-Pad1)
- J8 pad 9: Net-(J8-Pad9) -> +5V
Routing:
- net +5V: track 0.00 -> 300.8 mm, vias 0 -> 22
- net +3V3: track 0.00 -> 298.2 mm, vias 0 -> 12
- net SCL_33: track 0.00 -> 183.8 mm, vias 0 -> 5
- net SDA_33: track 0.00 -> 178.7 mm, vias 0 -> 6
- net +3.3VA: track 0.00 -> 156.3 mm, vias 0 -> 4
- net +BATT: track 0.00 -> 100.6 mm
- net GND: track 0.00 -> 78.3 mm, vias 0 -> 7
- net prez: track 0.00 -> 74.3 mm, vias 0 -> 4
- net SCL_5: track 0.00 -> 70.5 mm, vias 0 -> 2
- net Rail1: track 0.00 -> 69.3 mm
- net Net-(D5-Pad1): track 0.00 -> 68.1 mm, vias 0 -> 4
- net Rail2: track 0.00 -> 64.1 mm
- net Net-(D7-Pad1): track 0.00 -> 64.0 mm, vias 0 -> 2
- net SDA_5: track 0.00 -> 63.2 mm, vias 0 -> 2
- net Net-(F3-Pad1): track 0.00 -> 59.5 mm
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- added copper zone on F.Cu, net +BATT
- added copper zone on B.Cu, net GND
- added copper zone on In1.Cu, net GND
- added copper zone on In2.Cu, net GND
- added copper zone on F.Cu, net Net-(F3-Pad1)
- added copper zone on F.Cu, net Net-(F3-Pad2)
Other:
- board size 67.3 x 75 mm -> 84.7 x 126.2 mm
- copper layers 2 -> 4
- rule pad_to_mask_clearance: 0.051 -> 0
- board text added: "+B"
- board text added: "3"
- board text added: "3v"
- board text added: "3v Fuse"
- board text added: "3v Reg"
- board text added: "5"
- board text added: "5V IO"
- board text added: "5v"
- board text added: "5v Fuse"
- board text added: "5v Reg"
- board text added: "B"
- board text added: "B E C"
- board text added: "BAT"
- board text added: "BEC1"
- board text added: "BEC2"
- board text added: "C"
- board text added: "CLK"
- board text added: "CMD"
- board text added: "D"
- board text added: "EN"
- board text added: "G"
- board text added: "GND"
- board text added: "IIC 3V"
- board text added: "IIC 5V"
- board text added: "IO1"
- board text added: "IO12"
- board text added: "IO13"
- board text added: "IO14"
- board text added: "IO15"
- board text added: "IO16"
- board text added: "IO17"
- board text added: "IO18"
- board text added: "IO19"
- board text added: "IO2"
- board text added: "IO21"
- board text added: "IO22"
- board text added: "IO23"
- board text added: "IO25"
- board text added: "IO26"
- board text added: "IO27"
- board text added: "IO32"
- board text added: "IO33"
- board text added: "IO34"
- board text added: "IO35"
- board text added: "IO4"
- board text added: "IO5"
- board text added: "L Bank Fuse"
- board text added: "L Bank Pow Select"
- board text added: "Main Fuse"
- board text added: "R Bank Fuse"
- board text added: "R Bank Pow Select"
- board text added: "RIB Rev6.1 Kalbi"
- board text added: "RX0"
- board text added: "SD0"
- board text added: "SD1"
- board text added: "SD2"
- board text added: "SD3"
- board text added: "SVN"
- board text added: "SVP"
- board text added: "TX0"
- board text added: "U"
